File: Kicad/SLAPS_Solar_Harvester/SLAPS_Solar_Harvester.kicad_pcb (KiCad board)
At the start: 2 copper layers, 67.5 x 34 mm, 58 parts, among them J1 USB_C_Receptacle_USB2.0, J2 Conn_01x01_Male, J3 Conn_01x01_Male, J4 Conn_01x01_Male, J5 Conn_01x01_Male, Q1 Q_NMOS_GSD, U1 ATSAMD21E18A-A, U2 MS5607-02BA, U3 AEM10941, U4 XTSD, U7 TPS7A0530PDBV, U8 LTC4419, Y1 ABS07-32.768KHZ-T

Commit message: working on RP2040 rev
Parts:
- removed TP12, TP13, TP14, TP15: TestPoint, TestPoint:TestPoint_Pad_D1.0mm
- removed TP16: SWCLK, TestPoint:TestPoint_Pad_D1.0mm
- removed TP17: SWDIO, TestPoint:TestPoint_Pad_D1.0mm
- removed U7: TPS7A0530PDBV, Package_TO_SOT_SMD:SOT-23-5
- removed U8: LTC4419, Package_SO:MSOP-12-1EP_3x4mm_P0.65mm_EP1.65x2.85mm_ThermalVias
- added B2: KMR2, Button_Switch_SMD:SW_Push_1P1T_NO_CK_KMR2, F.Cu at (168.2, 93.3)
- added C10: 1uF, Capacitor_SMD:C_0402_1005Metric_Pad0.74x0.62mm_HandSolder, F.Cu at (160.1, 100.7)
- added C11: 100nF, Capacitor_SMD:C_0402_1005Metric_Pad0.74x0.62mm_HandSolder, F.Cu at (156.1, 100.7)
- added C12: 100nF, Capacitor_SMD:C_0402_1005Metric_Pad0.74x0.62mm_HandSolder, F.Cu at (158.3, 100.7)
- added C13: 100nF, Capacitor_SMD:C_0402_1005Metric_Pad0.74x0.62mm_HandSolder, F.Cu at (157.2, 100.7)
- added C14: 100nF, Capacitor_SMD:C_0603_1608Metric_Pad1.08x0.95mm_HandSolder, B.Cu at (169.3, 108.9)
- added C15: 1uF, Capacitor_SMD:C_0603_1608Metric_Pad1.08x0.95mm_HandSolder, B.Cu at (167.2, 93.8)
- added C16: 1uF, Capacitor_SMD:C_0603_1608Metric_Pad1.08x0.95mm_HandSolder, B.Cu at (163.9, 96.4)
- added C17: 2.2uF, Capacitor_SMD:C_0603_1608Metric_Pad1.08x0.95mm_HandSolder, B.Cu at (131.2, 115.5)
- added C18: 10uF, Capacitor_SMD:C_0603_1608Metric_Pad1.08x0.95mm_HandSolder, B.Cu at (129.5, 107.0)
- added C19: 0.1uF, Capacitor_SMD:C_0603_1608Metric_Pad1.08x0.95mm_HandSolder, B.Cu at (159.4, 113.7)
- added C20: 10uF, Capacitor_SMD:C_0603_1608Metric_Pad1.08x0.95mm_HandSolder, F.Cu at (153.7, 99.7)
- added J6: SOICbite, Connector:SOIC_clipProgSmall, F.Cu at (150.0, 90.4)
- added R10: 715k, Resistor_SMD:R_0603_1608Metric_Pad0.98x0.95mm_HandSolder, B.Cu at (127.5, 112.5)
- added R11: 585, Resistor_SMD:R_0603_1608Metric_Pad0.98x0.95mm_HandSolder, F.Cu at (208.5, 156.3)
- added R12: 10k, Resistor_SMD:R_0603_1608Metric_Pad0.98x0.95mm_HandSolder, B.Cu at (153.1, 111.8)
- added R13: 10k, Resistor_SMD:R_0603_1608Metric_Pad0.98x0.95mm_HandSolder, B.Cu at (153.1, 113.4)
- added R8: 5.1k, Resistor_SMD:R_0603_1608Metric_Pad0.98x0.95mm_HandSolder, F.Cu at (181.6, 98.5)
- added R9: 1M, Resistor_SMD:R_0603_1608Metric_Pad0.98x0.95mm_HandSolder, B.Cu at (125.8, 112.5)
- added U5: AEM10941, Package_DFN_QFN:QFN-28-1EP_5x5mm_P0.5mm_EP3.35x3.35mm_ThermalVias, B.Cu at (135.5, 103.4)
- added U6: MS5607-02BA, Package_LGA:LGA-8_3x5mm_P1.25mm, B.Cu at (156.7, 113.6)
- B1: value SW_Push -> KMR2; footprint Button_Switch_SMD:SW_SPST_EVQQ2 -> Button_Switch_SMD:SW_Push_1P1T_NO_CK_KMR2
- C1: value 1uF -> C_Small
- C2: value 0.1uF -> C_Small
- C3: value 0.1uF -> 100nF; footprint Capacitor_SMD:C_0603_1608Metric_Pad1.08x0.95mm_HandSolder -> Capacitor_SMD:C_0402_1005Metric_Pad0.74x0.62mm_HandSolder; moved to F.Cu
- C4, C5: value 1uF -> 100nF; footprint Capacitor_SMD:C_0603_1608Metric_Pad1.08x0.95mm_HandSolder -> Capacitor_SMD:C_0402_1005Metric_Pad0.74x0.62mm_HandSolder; moved to F.Cu
- C6: value 2.2uF -> 100nF; footprint Capacitor_SMD:C_0603_1608Metric_Pad1.08x0.95mm_HandSolder -> Capacitor_SMD:C_0402_1005Metric_Pad0.74x0.62mm_HandSolder; moved to F.Cu
- C7: value 10uF -> 100nF; footprint Capacitor_SMD:C_0603_1608Metric_Pad1.08x0.95mm_HandSolder -> Capacitor_SMD:C_0402_1005Metric_Pad0.74x0.62mm_HandSolder; moved to F.Cu
- C8: value 22pF -> 1uF; footprint Capacitor_SMD:C_0603_1608Metric_Pad1.08x0.95mm_HandSolder -> Capacitor_SMD:C_0402_1005Metric_Pad0.74x0.62mm_HandSolder; moved to F.Cu
- C9: value 22pF -> 100nF; footprint Capacitor_SMD:C_0603_1608Metric_Pad1.08x0.95mm_HandSolder -> Capacitor_SMD:C_0402_1005Metric_Pad0.74x0.62mm_HandSolder; moved to F.Cu
- D1: value LED -> USBLC6-2SC6; footprint Diode_SMD:D_0603_1608Metric_Pad1.05x0.95mm_HandSolder -> Package_TO_SOT_SMD_AKL:SOT-23-6; moved to B.Cu
- D2: value USBLC6-2SC6 -> LED; footprint Package_TO_SOT_SMD_AKL:SOT-23-6 -> Diode_SMD:D_0603_1608Metric_Pad1.05x0.95mm_HandSolder; moved to F.Cu
- F1: footprint Fuse:Fuse_1210_3225Metric_Pad1.42x2.65mm_HandSolder -> Fuse:Fuse_0805_2012Metric_Pad1.15x1.40mm_HandSolder
- JP1, JP2, TP6, TP7: moved to F.Cu
- R1: value 5.1k -> 1k
- R2: value 5.1k -> 10k; moved to F.Cu
- R3, R4: value 10k -> 27
- R5: value 1M -> 1k
- R6: value 715k -> 10k
- R7: value 585 -> 5.1k
- U1: value ATSAMD21E18A-A -> RP2040; footprint Package_QFP:TQFP-32_7x7mm_P0.8mm -> RP2040_minimal:RP2040-QFN-56
- U2: value MS5607-02BA -> W25Q128JVS; footprint Package_LGA:LGA-8_3x5mm_P1.25mm -> Package_SO:SOIC-8_5.23x5.23mm_P1.27mm
- U3: value AEM10941 -> TPS7A0530PDBV; footprint Package_DFN_QFN:QFN-28-1EP_5x5mm_P0.5mm_EP3.35x3.35mm_ThermalVias -> Package_TO_SOT_SMD:SOT-23-5
- U4: value XTSD -> LTC4419; footprint Package_LGA:LGA-8_XTSD -> Package_SO:MSOP-12-1EP_3x4mm_P0.65mm_EP1.65x2.85mm_ThermalVias
- Y1: value ABS07-32.768KHZ-T -> 445I23D12M00000; footprint Crystal:ABS07-32.768KHZ-T -> Crystal:Crystal_SMD_5032-2Pin_5.0x3.2mm_HandSoldering
- moved JP1 85.9 mm to (200.5, 144.5), turned to 0 degrees
- moved TP7 80.2 mm to (105.3, 110.1), turned to 0 degrees
- moved JP2 79.5 mm to (203.0, 136.0), turned to 0 degrees
- moved Q1 77.8 mm to (207.9, 153.0), turned to 0 degrees
- moved TP4 77.7 mm to (105.5, 104.0)
- moved D2 71.3 mm to (208.1, 158.5), turned to 0 degrees
- moved R6 46.1 mm to (170.3, 112.8), turned to 180 degrees
- moved R5 45.9 mm to (170.3, 114.4), turned to 180 degrees
- moved TP10 39.5 mm to (116.7, 99.0), turned to 0 degrees
- moved TP6 39.1 mm to (108.5, 104.0), turned to 0 degrees
- moved U3 32.4 mm to (166.8, 96.4), turned to 180 degrees
- moved TP5 28.5 mm to (127.6, 116.8), turned to 180 degrees
- moved C6 28.0 mm to (154.1, 103.8)
- moved C7 27.1 mm to (159.7, 106.4), turned to 90 degrees
- moved TP8 23.2 mm to (153.7, 115.4)
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Connections:
- B1 pad 1: Net-(B1-Pad1) -> GND
- B1 pad 2: GND -> Net-(B1-Pad2)
- C1 pad 1: Net-(C1-Pad1) -> GND
- C1 pad 2: GND -> Net-(C1-Pad2)
- C2 pad 1: +3V3 -> GND
- C2 pad 2: GND -> Net-(C2-Pad2)
- C3 pad 1: +3V3 -> +1V1
- C4 pad 1: VBUS -> +1V1
- C5 pad 1: +3V0 -> +3V3
- C6 pad 1: +3V0 -> +3V3
- C7 pad 1: /VSRC -> +3V3
- C8 pad 1: Net-(C8-Pad1) -> +1V1
- C8 pad 2: Net-(C8-Pad2) -> GND
- C9 pad 1: Net-(C9-Pad1) -> +3V3
- C9 pad 2: Net-(C9-Pad2) -> GND
- D1 pad 1: GND -> /USB_D+
- D1 pad 2: Net-(D1-Pad2) -> GND
- D2 pad 1: /D- -> GND
- D2 pad 2: GND -> Net-(D2-Pad2)
- J1 pad A6: Net-(D2-Pad6) -> Net-(D1-Pad6)
- J1 pad A7: Net-(D2-Pad4) -> Net-(D1-Pad4)
- J1 pad B6: Net-(D2-Pad6) -> Net-(D1-Pad6)
- J1 pad B7: Net-(D2-Pad4) -> Net-(D1-Pad4)
- J1 pad S1: GND -> unconnected-(J1-PadS1)
- R1 pad 1: Net-(J1-PadB5) -> Net-(C2-Pad2)
- R1 pad 2: GND -> Net-(R1-Pad2)
- R2 pad 1: Net-(J1-PadA5) -> +3V3
- R2 pad 2: GND -> Net-(B1-Pad2)
- R3 pad 1: +3V3 -> Net-(R3-Pad1)
- R3 pad 2: /SCL -> /USB_D+
- R4 pad 1: +3V3 -> Net-(R4-Pad1)
- R4 pad 2: /SDA -> /USB_D-
- R5 pad 1: +3V0 -> Net-(B2-Pad2)
- R5 pad 2: Net-(R5-Pad2) -> /QSPI_SS
- R6 pad 1: Net-(R5-Pad2) -> +3V3
- R6 pad 2: GND -> /QSPI_SS
- R7 pad 1: Net-(Q1-Pad2) -> Net-(J1-PadA5)
- R7 pad 2: Net-(D1-Pad2) -> GND
- TP10 pad 1: /SSEL -> +3V3
- TP11 pad 1: /SCK -> +1V8
- TP2 pad 1: Net-(D2-Pad6) -> /USB_D+
- TP3 pad 1: Net-(D2-Pad4) -> /USB_D-
- TP5 pad 1: /SCL -> +3V0
- TP6 pad 1: /SDA -> /VSRC
- TP7 pad 1: +3V0 -> /VBUCK
- TP8 pad 1: /VBUCK -> /SDA
- TP9 pad 1: /VSRC -> /SCL
- U1 pad 1: Net-(C8-Pad1) -> +3V3
- U1 pad 10: GND -> +3V3
- U1 pad 12: /MISO -> unconnected-(U1-Pad12)
- U1 pad 13: /MOSI -> unconnected-(U1-Pad13)
- U1 pad 14: /SCK -> unconnected-(U1-Pad14)
- U1 pad 15: /SSEL -> unconnected-(U1-Pad15)
- U1 pad 19: unconnected-(U1-Pad19) -> GND
- U1 pad 2: Net-(C9-Pad1) -> unconnected-(U1-Pad2)
- U1 pad 20: unconnected-(U1-Pad20) -> Net-(C1-Pad2)
- U1 pad 21: /D1 -> Net-(R1-Pad2)
- U1 pad 22: unconnected-(U1-Pad22) -> +3V3
- U1 pad 23: /D- -> +1V1
- U1 pad 24: /D+ -> /SWCLK
- U1 pad 25: unconnected-(U1-Pad25) -> /SWDIO
- U1 pad 26: Net-(B1-Pad1) -> Net-(B1-Pad2)
- U1 pad 28: GND -> unconnected-(U1-Pad28)
- U1 pad 29: Net-(C1-Pad1) -> unconnected-(U1-Pad29)
- U1 pad 30: +1V8 -> unconnected-(U1-Pad30)
- U1 pad 31: Net-(TP16-Pad1) -> unconnected-(U1-Pad31)
- U1 pad 32: Net-(TP17-Pad1) -> unconnected-(U1-Pad32)
- U1 pad 4: unconnected-(U1-Pad4) -> /SDA
- U1 pad 6: /SDA -> unconnected-(U1-Pad6)
- U1 pad 8: unconnected-(U1-Pad8) -> /D1
- U1 pad 9: +1V8 -> unconnected-(U1-Pad9)
- U2 pad 1: +3V3 -> /QSPI_SS
- U2 pad 2: +3V3 -> /QSPI_SD1
- U2 pad 3: GND -> /QSPI_SD2
- U2 pad 5: GND -> /QSPI_SD0
- U2 pad 6: unconnected-(U2-Pad6) -> /QSPI_SCLK
- U2 pad 7: /SDA -> /QSPI_SD3
- U2 pad 8: /SCL -> +3V3
- U3 pad 1: Net-(CBOOST1-Pad1) -> VBUS
- U3 pad 2: Net-(LBUCK1-Pad2) -> GND
- U3 pad 3: /VBUCK -> VBUS
- U3 pad 4: /VBUCK -> unconnected-(U3-Pad4)
- U3 pad 5: /VBUCK -> +3V0
- U4 pad 1: unconnected-(U4-Pad1) -> +3V0
- U4 pad 2: /SSEL -> unconnected-(U4-Pad2)
- U4 pad 3: /SCK -> GND
- U4 pad 4: GND -> Net-(R10-Pad1)
- U4 pad 5: /MOSI -> GND
- U4 pad 6: /MISO -> unconnected-(U4-Pad6)
- U4 pad 8: +3V3 -> unconnected-(U4-Pad8)
- Y1 pad 1: Net-(C9-Pad2) -> Net-(C2-Pad2)
- Y1 pad 2: Net-(C8-Pad2) -> Net-(C1-Pad2)
Routing:
- net Net-(J4-Pad1): track 129.7 -> 33.2 mm
- net +3V3: track 24.2 -> 83.2 mm, vias 4 -> 9
- net Net-(B2-Pad2): track 0.00 -> 47.2 mm, vias 0 -> 1
- net +3V0: track 94.7 -> 61.9 mm, vias 0 -> 2
- net Net-(B1-Pad1): track 30.2 -> 0.00 mm, vias 3 -> 0
- net /VBUCK: track 0.00 -> 29.9 mm, vias 0 -> 2
- net +1V8: track 29.9 -> 3.43 mm, vias 2 -> 1
- net /QSPI_SS: track 0.00 -> 21.2 mm
- net Net-(B1-Pad2): track 0.00 -> 19.9 mm, vias 0 -> 1
- net /MISO: track 16.0 -> 0.00 mm, vias 1 -> 0
- net /QSPI_SD1: track 0.00 -> 15.0 mm
- net /USB_D+: track 0.00 -> 14.1 mm
- net /SWCLK: track 0.00 -> 13.9 mm, vias 0 -> 1
- net /SSEL: track 13.2 -> 0.00 mm, vias 1 -> 0
- net /MOSI: track 13.1 -> 0.00 mm, vias 1 -> 0
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- removed copper zone on B.Cu, net +3V3
- removed copper zone on B.Cu, net /VBUCK
- removed copper zone on B.Cu, net /VSRC
- removed copper zone on B.Cu, net Net-(R5-Pad2)
- removed copper zone on F.Cu, net VBUS
Other:
- outline, holes or cut-outs redrawn
- board text removed: "RESET"
- board text removed: "SLAPS-SH"
- board text removed: "V1.0"
- board text removed: "designed with love by the SLAPS team"

Commit message: some extras
Parts:
- TP10, TP6, TP7: moved to B.Cu
- TP4: footprint TestPoint:TestPoint_Pad_D1.0mm -> TestPoint:TestPoint_Keystone_5000-5004_Miniature
- Y1: footprint Crystal:Crystal_SMD_5032-2Pin_5.0x3.2mm_HandSoldering -> Crystal:Crystal_SMD_5032-2Pin_5.0x3.2mm
- moved JP1 81.8 mm to (135.8, 94.5), turned to 180 degrees
- moved TP4 79.5 mm to (184.3, 114.3)
- moved JP2 75.0 mm to (140.5, 94.5)
- moved D2 54.4 mm to (185.0, 109.3), turned to -90 degrees
- moved R11 53.3 mm to (183.4, 109.3), turned to -90 degrees
- moved Q1 51.6 mm to (180.5, 109.3), turned to 180 degrees
- moved TP7 33.6 mm to (136.5, 97.4), turned to 180 degrees
- moved TP10 24.2 mm to (139.9, 105.7), turned to 180 degrees
- moved TP6 23.6 mm to (132.0, 107.1), turned to 180 degrees
- moved C5 3.86 mm to (163.9, 103.6), turned to 0 degrees
- moved J2 2.55 mm to (124.8, 96.7)
- moved C2 1.80 mm to (148.1, 103.4)
- moved C1 1.80 mm to (150.3, 109.7)
- moved R1 1.80 mm to (150.3, 106.2)
- moved TP3 1.56 mm to (168.1, 101.8)
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Routing:
- net Net-(J4-Pad1): track 33.2 -> 106.8 mm
- net /D1: track 0.00 -> 46.3 mm, vias 0 -> 1
- net /VBUCK: track 29.9 -> 47.4 mm
- net +3V3: track 83.2 -> 70.1 mm, vias 9 -> 10
- net Net-(JP1-Pad2): track 0.00 -> 9.85 mm, vias 0 -> 1
- net Net-(JP2-Pad2): track 1.40 -> 9.53 mm
- net Net-(BT1-Pad1): track 0.00 -> 7.77 mm
- net Net-(C2-Pad2): track 0.00 -> 5.71 mm
- net GND: track 58.6 -> 53.5 mm, vias 10 -> 29
- net +1V1: track 12.5 -> 17.3 mm
- net Net-(Q1-Pad2): track 0.00 -> 1.78 mm
- net Net-(D2-Pad2): track 0.00 -> 1.62 mm
- net /VSRC: track 7.60 -> 9.02 mm
- net Net-(B2-Pad2): track 47.2 -> 46.1 mm
- net /SWDIO: track 12.9 -> 12.4 mm
- added copper zone on F.Cu, net +1V1
- added copper zone on B.Cu, net +3V3
- added copper zone on B.Cu, net GND

Commit message: more work on V1.1
Parts:
- C1, C2: value C_Small -> 27pF
- C19: value 0.1uF -> 100nF
- R11: value 585 -> 590
Changed lines of the file:
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@@
       (effects (font (size 0.5 0.5) (thickness 0.125)))
     )
-    (fp_text value "585" (at 0 1.43 90) (layer "F.Fab")
+    (fp_text value "590" (at 0 1.43 90) (layer "F.Fab")
       (effects (font (size 1 1) (thickness 0.15)))
     )
@@
     (fp_line (start -1.5 -0.56) (end 7.45 -0.56) (layer "F.Fab") (width 0.1))
     (fp_line (start -1.5 8.61) (end 7.45 8.61) (layer "F.Fab") (width 0.1))
-    (pad "A1" thru_hole circle (at 0 0 180) (size 0.7 0.7) (drill 0.4) (layers *.Cu *.Mask)
+    (pad "A1" thru_hole circle (at 0 0 180) (size 0.67 0.67) (drill 0.4) (layers *.Cu *.Mask)
       (net 33 "GND") (pinfunction "GND") (pintype "passive"))
-    (pad "A4" thru_hole circle (at 0.85 0 180) (size 0.7 0.7) (drill 0.4) (layers *.Cu *.Mask)
+    (pad "A4" thru_hole circle (at 0.85 0 180) (size 0.67 0.67) (drill 0.4) (layers *.Cu *.Mask)
       (net 29 "VBUS") (pinfunction "VBUS") (pintype "power_out"))
-    (pad "A5" thru_hole circle (at 1.7 0 180) (size 0.7 0.7) (drill 0.4) (layers *.Cu *.Mask)
+    (pad "A5" thru_hole circle (at 1.7 0 180) (size 0.67 0.67) (drill 0.4) (layers *.Cu *.Mask)
       (net 21 "Net-(J1-PadA5)") (pinfunction "CC1") (pintype "bidirectional"))
-    (pad "A6" thru_hole circle (at 2.55 0 180) (size 0.7 0.7) (drill 0.4) (layers *.Cu *.Mask)
+    (pad "A6" thru_hole circle (at 2.55 0 180) (size 0.67 0.67) (drill 0.4) (layers *.Cu *.Mask)
       (net 19 "Net-(D1-Pad6)") (pinfunction "D+") (pintype "bidirectional"))
-    (pad "A7" thru_hole circle (at 3.4 0 180) (size 0.7 0.7) (drill 0.4) (layers *.Cu *.Mask)
+    (pad "A7" thru_hole circle (at 3.4 0 180) (size 0.67 0.67) (drill 0.4) (layers *.Cu *.Mask)
       (net 91 "Net-(D1-Pad4)") (pinfunction "D-") (pintype "bidirectional"))
-    (pad "A8" thru_hole circle (at 4.25 0 180) (size 0.7 0.7) (drill 0.4) (layers *.Cu *.Mask)
+    (pad "A8" thru_hole circle (at 4.25 0 180) (size 0.67 0.67) (drill 0.4) (layers *.Cu *.Mask)
       (net 22 "unconnected-(J1-PadA8)") (pinfunction "SBU1") (pintype "bidirectional+no_connect"))
-    (pad "A9" thru_hole circle (at 5.1 0 180) (size 0.7 0.7) (drill 0.4) (layers *.Cu *.Mask)
+    (pad "A9" thru_hole circle (at 5.1 0 180) (size 0.67 0.67) (drill 0.4) (layers *.Cu *.Mask)
       (net 29 "VBUS") (pinfunction "VBUS") (pintype "passive"))
-    (pad "A12" thru_hole circle (at 5.95 0 180) (size 0.7 0.7) (drill 0.4) (layers *.Cu *.Mask)
+    (pad "A12" thru_hole circle (at 5.95 0 180) (size 0.67 0.67) (drill 0.4) (layers *.Cu *.Mask)
       (net 33 "GND") (pinfunction "GND") (pintype "passive"))
-    (pad "B1" thru_hole circle (at 5.95 1.35 180) (size 0.7 0.7) (drill 0.4) (layers *.Cu *.Mask)
+    (pad "B1" thru_hole circle (at 5.95 1.35 180) (size 0.67 0.67) (drill 0.4) (layers *.Cu *.Mask)
       (net 33 "GND") (pinfunction "GND") (pintype "passive"))
-    (pad "B4" thru_hole circle (at 5.1 1.35 180) (size 0.7 0.7) (drill 0.4) (layers *.Cu *.Mask)
+    (pad "B4" thru_hole circle (at 5.1 1.35 180) (size 0.67 0.67) (drill 0.4) (layers *.Cu *.Mask)
       (net 29 "VBUS") (pinfunction "VBUS") (pintype "passive"))
-    (pad "B5" thru_hole circle (at 4.25 1.35 180) (size 0.7 0.7) (drill 0.4) (layers *.Cu *.Mask)
+    (pad "B5" thru_hole circle (at 4.25 1.35 180) (size 0.67 0.67) (drill 0.4) (layers *.Cu *.Mask)
       (net 26 "Net-(J1-PadB5)") (pinfunction "CC2") (pintype "bidirectional"))
-    (pad "B6" thru_hole circle (at 3.4 1.35 180) (size 0.7 0.7) (drill 0.4) (layers *.Cu *.Mask)
+    (pad "B6" thru_hole circle (at 3.4 1.35 180) (size 0.67 0.67) (drill 0.4) (layers *.Cu *.Mask)
       (net 19 "Net-(D1-Pad6)") (pinfunction "D+") (pintype "bidirectional"))
-    (pad "B7" thru_hole circle (at 2.55 1.35 180) (size 0.7 0.7) (drill 0.4) (layers *.Cu *.Mask)
+    (pad "B7" thru_hole circle (at 2.55 1.35 180) (size 0.67 0.67) (drill 0.4) (layers *.Cu *.Mask)
       (net 91 "Net-(D1-Pad4)") (pinfunction "D-") (pintype "bidirectional"))
-    (pad "B8" thru_hole circle (at 1.7 1.35 180) (size 0.7 0.7) (drill 0.4) (layers *.Cu *.Mask)
+    (pad "B8" thru_hole circle (at 1.7 1.35 180) (size 0.67 0.67) (drill 0.4) (layers *.Cu *.Mask)
       (net 28 "unconnected-(J1-PadB8)") (pinfunction "SBU2") (pintype "bidirectional+no_connect"))
-    (pad "B9" thru_hole circle (at 0.85 1.35 180) (size 0.7 0.7) (drill 0.4) (layers *.Cu *.Mask)
+    (pad "B9" thru_hole circle (at 0.85 1.35 180) (size 0.67 0.67) (drill 0.4) (layers *.Cu *.Mask)
       (net 29 "VBUS") (pinfunction "VBUS") (pintype "passive"))
-    (pad "B12" thru_hole circle (at 0 1.35 180) (size 0.7 0.7) (drill 0.4) (layers *.Cu *.Mask)
+    (pad "B12" thru_hole circle (at 0 1.35 180) (size 0.67 0.67) (drill 0.4) (layers *.Cu *.Mask)
       (net 33 "GND") (pinfunction "GND") (pintype "passive"))
     (pad "S1" thru_hole oval (at 7.3 0.98 180) (size 0.9 2.4) (drill oval 0.6 2.1) (layers *.Cu *.Mask)
@@
       (effects (font (size 0.5 0.5) (thickness 0.125)) (justify mirror))
     )
-    (fp_text value "0.1uF" (at 0 -1.43 90) (layer "B.Fab")
+    (fp_text value "100nF" (at 0 -1.43 90) (layer "B.Fab")
       (effects (font (size 1 1) (thickness 0.15)) (justify mirror))
     )
@@
       (effects (font (size 0.5 0.5) (thickness 0.125)) (justify mirror))
     )
-    (fp_text value "C_Small" (at 0 -1.43 90) (layer "B.Fab")
+    (fp_text value "27pF" (at 0 -1.43 90) (layer "B.Fab")
       (effects (font (size 1 1) (thickness 0.15)) (justify mirror))
     )
@@
       (effects (font (size 0.5 0.5) (thickness 0.125)) (justify mirror))
     )
-    (fp_text value "C_Small" (at 0 -1.43) (layer "B.Fab")
+    (fp_text value "27pF" (at 0 -1.43) (layer "B.Fab")
       (effects (font (size 1 1) (thickness 0.15)) (justify mirror))
     )
@@
   (via (at 136.3 108) (size 0.8) (drill 0.4) (layers "F.Cu" "B.Cu") (free) (net 34))
   (via (at 137 107.3) (size 0.8) (drill 0.4) (layers "F.Cu" "B.Cu") (free) (net 34))
-  (segment (start 184.5 99.8) (end 172.8 111.5) (width 0.25) (layer "F.Cu") (net 35))
-  (segment (start 184.5 94.9) (end 184.5 99.8) (width 0.25) (layer "F.Cu") (net 35))
+  (segment (start 184.5 99.8) (end 172.8 111.5) (width 1) (layer "F.Cu") (net 35))
+  (segment (start 184.5 94.9) (end 184.5 99.8) (width 1) (layer "F.Cu") (net 35))
   (segment (start 169 91.25) (end 169 95.35) (width 1) (layer "F.Cu") (net 35))
   (segment (start 180.85 91.25) (end 181.95 92.35) (width 1) (layer "F.Cu") (net 35))
   (segment (start 169 91.25) (end 180.85 91.25) (width 1) (layer "F.Cu") (net 35))
-  (segment (start 181.95 92.35) (end 184.5 94.9) (width 0.25) (layer "F.Cu") (net 35))
+  (segment (start 181.95 92.35) (end 184.5 94.9) (width 1) (layer "F.Cu") (net 35))
   (via (at 172.8 111.5) (size 0.8) (drill 0.4) (layers "F.Cu" "B.Cu") (net 35))
   (segment (start 172.8 112.8125) (end 172.8 111.5) (width 0.25) (layer "B.Cu") (net 35))

Commit message: more V1.1
Parts:
- added G***: LOGO, KiCAD Artwork:Warning, F.Cu at (156.8, 117.4)
- added REF**: BalloonArt, KiCAD Artwork:BalloonArt, F.Cu at (148.1, 102.2)
- moved TP4 12.7 mm to (186.2, 101.7)
Other:
- outline, holes or cut-outs redrawn
- board text added: "PLEASE READ! There's no polarity protection (I know) so double check the battery before you insert it. Fire is BAD!"
- board text added: "SLAPS-SH"
- board text added: "V1.1"
- board text added: "fingers crossed"
