File: Kicad/SLAPS_Solar_Harvester/SLAPS_Solar_Harvester.kicad_sch (KiCad schematic)
At the start: 58 parts, among them J1 USB_C_Receptacle_USB2.0, J2 Conn_01x01_Male, J3 Conn_01x01_Male, J4 Conn_01x01_Male, J5 Conn_01x01_Male, Q1 Q_NMOS_GSD, U1 ATSAMD21E18A-A, U2 MS5607-02BA, U3 AEM10941, U4 XTSD, U7 TPS7A0530PDBV, U8 LTC4419, Y1 ABS07-32.768KHZ-T

Commit message: started on V1.1
Parts:
- removed C3: 0.1uF, Capacitor_SMD:C_0603_1608Metric_Pad1.08x0.95mm_HandSolder, symbol Device:C_Small
- removed C4, C5: 1uF, Capacitor_SMD:C_0603_1608Metric_Pad1.08x0.95mm_HandSolder, symbol Device:C_Small
- removed C6: 2.2uF, Capacitor_SMD:C_0603_1608Metric_Pad1.08x0.95mm_HandSolder, symbol Device:C_Small
- removed C7: 10uF, Capacitor_SMD:C_0603_1608Metric_Pad1.08x0.95mm_HandSolder, symbol Device:C_Small
- removed C9: 22pF, Capacitor_SMD:C_0603_1608Metric_Pad1.08x0.95mm_HandSolder, symbol Device:C_Small
- removed D1: LED, Diode_SMD:D_0603_1608Metric_Pad1.05x0.95mm_HandSolder, symbol Device:LED
- removed D2: USBLC6-2SC6, Package_TO_SOT_SMD_AKL:SOT-23-6, symbol Diode_TVS_AKL:USBLC6-2SC6
- removed TP12, TP13, TP14, TP15: TestPoint, TestPoint:TestPoint_Pad_D1.0mm, symbol Connector:TestPoint
- removed TP16: SWCLK, TestPoint:TestPoint_Pad_D1.0mm, symbol Connector:TestPoint
- removed TP17: SWDIO, TestPoint:TestPoint_Pad_D1.0mm, symbol Connector:TestPoint
- removed U1: ATSAMD21E18A-A, Package_QFP:TQFP-32_7x7mm_P0.8mm, symbol MCU_Microchip_SAMD:ATSAMD21E18A-A
- removed U2: MS5607-02BA, Package_LGA:LGA-8_3x5mm_P1.25mm, symbol Sensor_Pressure:MS5607-02BA
- removed U3: AEM10941, Package_DFN_QFN:QFN-28-1EP_5x5mm_P0.5mm_EP3.35x3.35mm_ThermalVias, symbol Battery_Management:AEM10941
- removed U4: XTSD, Package_LGA:LGA-8_XTSD, symbol Memory_Flash:XTSD
- removed U7: TPS7A0530PDBV, Package_TO_SOT_SMD:SOT-23-5, symbol Regulator_Linear:TPS7A0530PDBV
- removed U8: LTC4419, Package_SO:MSOP-12-1EP_3x4mm_P0.65mm_EP1.65x2.85mm_ThermalVias, symbol Power_Management:LTC4419
- added B2: KMR2, symbol Switch:SW_Push
- added C10: 1uF, symbol Device:C_Small
- added C14, C? (x9): 100nF, symbol Device:C_Small
- added C15, C16: 1uF, Capacitor_SMD:C_0603_1608Metric_Pad1.08x0.95mm_HandSolder, symbol Device:C_Small
- added C17: 2.2uF, Capacitor_SMD:C_0603_1608Metric_Pad1.08x0.95mm_HandSolder, symbol Device:C_Small
- added C18: 10uF, Capacitor_SMD:C_0603_1608Metric_Pad1.08x0.95mm_HandSolder, symbol Device:C_Small
- added C19: 0.1uF, Capacitor_SMD:C_0603_1608Metric_Pad1.08x0.95mm_HandSolder, symbol Device:C_Small
- added C?: 10uF, symbol Device:C_Small
- added D1: USBLC6-2SC6, Package_TO_SOT_SMD_AKL:SOT-23-6, symbol Diode_TVS_AKL:USBLC6-2SC6
- added D2: LED, Diode_SMD:D_0603_1608Metric_Pad1.05x0.95mm_HandSolder, symbol Device:LED
- added J6: SOICbite, symbol Connector:Conn_01x08_Female
- added R10: 715k, Resistor_SMD:R_0603_1608Metric_Pad0.98x0.95mm_HandSolder, symbol Device:R_Small
- added R11: 585, Resistor_SMD:R_0603_1608Metric_Pad0.98x0.95mm_HandSolder, symbol Device:R_Small
- added R12, R13: 10k, Resistor_SMD:R_0603_1608Metric_Pad0.98x0.95mm_HandSolder, symbol Device:R_Small
- added R8: 5.1k, Resistor_SMD:R_0603_1608Metric_Pad0.98x0.95mm_HandSolder, symbol Device:R_Small
- added R9: 1M, Resistor_SMD:R_0603_1608Metric_Pad0.98x0.95mm_HandSolder, symbol Device:R_Small
- added U1: RP2040, RP2040_minimal:RP2040-QFN-56, symbol MCU_RaspberryPi_RP2040:RP2040
- added U2: W25Q128JVS, Package_SO:SOIC-8_5.23x5.23mm_P1.27mm, symbol Memory_Flash:W25Q128JVS
- added U3: TPS7A0530PDBV, Package_TO_SOT_SMD:SOT-23-5, symbol Regulator_Linear:TPS7A0530PDBV
- added U4: LTC4419, Package_SO:MSOP-12-1EP_3x4mm_P0.65mm_EP1.65x2.85mm_ThermalVias, symbol Power_Management:LTC4419
- added U5: AEM10941, Package_DFN_QFN:QFN-28-1EP_5x5mm_P0.5mm_EP3.35x3.35mm_ThermalVias, symbol Battery_Management:AEM10941
- added U6: MS5607-02BA, Package_LGA:LGA-8_3x5mm_P1.25mm, symbol Sensor_Pressure:MS5607-02BA
- B1: value SW_Push -> KMR2; footprint Button_Switch_SMD:SW_SPST_EVQQ2 -> (none)
- C1: value 1uF -> C_Small; footprint Capacitor_SMD:C_0603_1608Metric_Pad1.08x0.95mm_HandSolder -> (none)
- C2: value 0.1uF -> C_Small; footprint Capacitor_SMD:C_0603_1608Metric_Pad1.08x0.95mm_HandSolder -> (none)
- C8: value 22pF -> 1uF; footprint Capacitor_SMD:C_0603_1608Metric_Pad1.08x0.95mm_HandSolder -> (none)
- R1: value 5.1k -> 1k; footprint Resistor_SMD:R_0603_1608Metric_Pad0.98x0.95mm_HandSolder -> (none)
- R2: value 5.1k -> 10k; footprint Resistor_SMD:R_0603_1608Metric_Pad0.98x0.95mm_HandSolder -> (none)
- R3, R4: value 10k -> 27; footprint Resistor_SMD:R_0603_1608Metric_Pad0.98x0.95mm_HandSolder -> (none)
- R5: value 1M -> 1k; footprint Resistor_SMD:R_0603_1608Metric_Pad0.98x0.95mm_HandSolder -> (none)
- R6: value 715k -> 10k; footprint Resistor_SMD:R_0603_1608Metric_Pad0.98x0.95mm_HandSolder -> (none)
- R7: value 585 -> 5.1k
- Y1: value ABS07-32.768KHZ-T -> 445I23D12M00000; footprint Crystal:ABS07-32.768KHZ-T -> (none)
Connections:
- net SCK is gone; now on net +1V8: TP11.1
- net SSEL is gone; now on net +3V3: TP10.1
- net +1V8: now also U5.11 (LVOUT)
- net +3V0: now also TP5.1, C16.1, C17.1, R9.1, U3.5 (OUT), U4.1 (V1); no longer R5.1, TP7.1
- net +3V3: now also R2.1, R6.1, C10.1, C14.1, C19.1, C?.1, C?.1, C?.1, C?.1, C?.1, C?.1, C?.1, C?.1, J6.1 (Pin_1), R12.1, R13.1, U1.1 (IOVDD), U1.10 (IOVDD), U1.22 (IOVDD), U1.33 (IOVDD), U1.42 (IOVDD), U1.43 (ADC_AVDD), U1.44 (VREG_IN), U1.48 (USB_VDD), U1.49 (IOVDD), U2.8 (VCC), U5.14 (HVOUT), U6.1 (VDD), U6.2 (PS); no longer C2.1, R3.1, R4.1
- net D1: now also U1.8 (GPIO6)
- net GND: now also B1.1, C1.1, C2.1, C8.2, R7.2, B2.1, C10.2, C14.2, C15.2, C16.2, C17.2, C18.2, C19.2, C?.2, C?.2, C?.2, C?.2, C?.2, C?.2, C?.2, C?.2, C?.2, C?.2, D1.2 (VN), D2.1 (K), J6.4 (Pin_4), R10.2, R8.2, U1.19 (TESTEN), U1.57 (GND), U2.4 (GND), U3.2 (GND), U4.10 (CMP2), U4.11 (NC), U4.13 (GND), U4.3 (CMP1), U4.5 (GND), U5.10 (FB_PRIM_U), U5.15 (BAL), U5.17 (PRIM), U5.29 (GND), U5.9 (FB_PRIM_D), U6.3 (GND), U6.4 (CSB), U6.5 (CSB); no longer B1.2, C1.2, C2.2, J1.S1 (SHIELD), R1.2, R2.2, R6.2
- net SCL: now also TP9.1, R12.2, U1.5 (GPIO3), U6.8 (SCLK); no longer R3.2, TP5.1
- net SDA: now also TP8.1, R13.2, U1.4 (GPIO2), U6.7 (SDI/SDA); no longer R4.2, TP6.1
- net VBUCK: now also TP7.1, U5.12 (ENHV), U5.18 (ENLV), U5.3 (BUCK), U5.4 (CFG[2]), U5.5 (CFG[1]), U5.6 (CFG[0]); no longer TP8.1
- net VBUS: now also C15.1, D1.5 (VP), U3.1 (IN), U3.3 (EN)
- net VSRC: now also TP6.1, C18.1, U4.9 (OUT), U5.25 (SRC), U5.26 (FB_COLD); no longer TP9.1
- net at J4.1 (Pin_1), J5.1 (Pin_1): now also U4.12 (V2)
- net at J1.A7 (D-), J1.B7 (D-): now also TP2.1, D1.4 (L2); no longer TP3.1
- net at J1.A6 (D+), J1.B6 (D+): now also TP3.1, D1.6 (L1); no longer TP2.1
- net at JP2.2 (C): now also U5.8 (SELMPP[0])
- net at CBOOST1.1: now also U5.1 (BOOST)
- net at CSRC1.1, LBOOST1.1: now also U5.27 (BUFSRC)
- net at R1.1: now also C2.2, Y1.1; no longer J1.B5 (CC2)
- net at J1.A5 (CC1): now also R7.1; no longer R2.1
- net at JP1.2 (C): now also U5.7 (SELMPP[1])
- net at F1.2: now also U5.16 (BATT)
- net +1V1: now reaches C8.1
- net +1V1: now also C?.1, C?.1, U1.23 (DVDD), U1.45 (VREG_VOUT), U1.50 (DVDD)
- net at Y1.2: now also C1.2, U1.20 (XIN); no longer C8.2
- net QSPI_SS: now reaches R5.2
- net QSPI_SS: now also R6.2, U1.56 (QSPI_SS), U2.1 (~{CS}); no longer R6.1
- net at LBUCK1.2: now also U5.2 (SWBUCK)
- net at LBOOST1.2: now also U5.28 (SWBOOST)
- net at Q1.2 (S): now also R11.1; no longer R7.1
- new net: R10.1, R9.2, U4.4 (ADJ)
- new net: R1.2, U1.21 (XOUT)
- new net: B1.2, R2.2, U1.26 (RUN)
- new net: D2.2 (A), R11.2
- new net: B2.2, R5.1
- new net: R4.1, U1.46 (USB_DM)
- new net: R3.1, U1.47 (USB_DP)
- new net: J1.B5 (CC2), R8.1
- new net QSPI_SCLK: U1.52 (QSPI_SCLK), U2.6 (CLK)
- new net QSPI_SD0: U1.53 (QSPI_SD0), U2.5 (DI(IO0))
- new net QSPI_SD1: U1.55 (QSPI_SD1), U2.2 (DO(IO1))
- new net QSPI_SD2: U1.54 (QSPI_SD2), U2.3 (IO2)
- new net QSPI_SD3: U1.51 (QSPI_SD3), U2.7 (IO3)
- new net SWCLK: J6.3 (Pin_3), U1.24 (SWCLK)
- new net SWDIO: J6.2 (Pin_2), U1.25 (SWD)
- new net USB_D+: D1.3 (L2), R3.2
- new net USB_D-: D1.1 (L1), R4.2
- no-connect marks 28 -> 45
Other:
- note added: "+3.0V selected due to optimal efficiency for AEM regulators"
- note added: "Flash"
- note added: "Make sure C10 is close to pin 44 of RP2040"
- note added: "Make sure C8 is close to pin 45 of RP2040"
- note added: "Make sure R3 and R4 are close to RP2040"
- note added: "SWD Header"
- note removed: "Storage"

Commit message: working on RP2040 rev
Parts:
- B1, B2: footprint (none) -> Button_Switch_SMD:SW_Push_1P1T_NO_CK_KMR2
- C1, C14, C2: footprint (none) -> Capacitor_SMD:C_0603_1608Metric_Pad1.08x0.95mm_HandSolder
- C10, C8: footprint (none) -> Capacitor_SMD:C_0402_1005Metric_Pad0.74x0.62mm_HandSolder
- C11, C12, C13, C3, C4, C5, C6, C7, C9: renamed from C?; footprint (none) -> Capacitor_SMD:C_0402_1005Metric_Pad0.74x0.62mm_HandSolder
- C20: renamed from C?; footprint (none) -> Capacitor_SMD:C_0603_1608Metric_Pad1.08x0.95mm_HandSolder
- F1: footprint Fuse:Fuse_1210_3225Metric_Pad1.42x2.65mm_HandSolder -> Fuse:Fuse_0805_2012Metric_Pad1.15x1.40mm_HandSolder
- J6: footprint (none) -> Connector:SOIC_clipProgSmall
- R1, R2, R3, R4, R5, R6: footprint (none) -> Resistor_SMD:R_0603_1608Metric_Pad0.98x0.95mm_HandSolder
- Y1: footprint (none) -> Crystal:Crystal_SMD_5032-2Pin_5.0x3.2mm_HandSoldering
Connections:
- net SWCLK: now also J6.2 (Pin_2); no longer J6.3 (Pin_3)
- net SWDIO: now also J6.3 (Pin_3); no longer J6.2 (Pin_2)
- net USB_D+: now also D1.1 (L1), TP2.1; no longer D1.3 (L2)
- net USB_D-: now also D1.3 (L2), TP3.1; no longer D1.1 (L1)
- net at D1.4 (L2), J1.A7 (D-), J1.B7 (D-): no longer TP2.1
- net at D1.6 (L1), J1.A6 (D+), J1.B6 (D+): no longer TP3.1
Other:
- note added: "DNF"
- moved on the sheet: BT1, C20, F1, TP2, TP3

Commit message: some extras
Parts:
- C1, C2: value C_Small -> 27pF
- C19: value 0.1uF -> 100nF
- R11: value 585 -> 590
- TP4: footprint TestPoint:TestPoint_Pad_D1.0mm -> TestPoint:TestPoint_Keystone_5000-5004_Miniature
- Y1: footprint Crystal:Crystal_SMD_5032-2Pin_5.0x3.2mm_HandSoldering -> Crystal:Crystal_SMD_5032-2Pin_5.0x3.2mm
Other:
- note added: "Never power AEM10941 without battery!!!"
- moved on the sheet: BT1, F1

Commit message: more work on V1.1
Other:
- moved on the sheet: C15, C16, J6, TP5, U3

Commit message: more V1.1
Changed lines of the file:
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@@
   (title_block
     (title "SLAPS Solar Harvester")
-    (date "2023-05-07")
+    (date "2023-05-17")
     (rev "V1.1")
     (company "Michael Shipman")
@@
     (effects (font (size 1.27 1.27) (thickness 0.254) bold) (justify left bottom))
   )
-  (text "Pressure & Temperature \nSensor" (at 201.93 168.91 0)
+  (text "Pressure & Temperature Sensor" (at 201.93 168.91 0)
     (effects (font (size 1.27 1.27) (thickness 0.254) bold) (justify left bottom))
   )
@@
     (effects (font (size 2.54 2.54) (thickness 0.508) bold) (justify right bottom))
   )
-  (text "Flash" (at 128.27 123.19 0)
+  (text "Flash" (at 128.27 124.46 0)
     (effects (font (size 2.54 2.54) (thickness 0.508) bold) (justify left bottom))
   )

Commit message: KiCad version 7
Parts:
- U1: symbol MCU_RaspberryPi_RP2040:RP2040 -> MCU_RaspberryPi:RP2040
Other:
- note added: "Solar Harvester/PMIC"
- note added: "This resistor ensure that we don't overdrive the LED"
- note added: "Transient Voltage Suppression"
- note removed: "Solar Harvester"

Commit message: Minimal firmware
Parts:
- C1, C2: value 27pF -> 22pF
- R1: value 1k -> DNP
Changed lines of the file:
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@@
     (stroke (width 0) (type dash))
   )
-  (polyline (pts (xy 139.7 33.02) (xy 198.12 33.02))
+  (polyline (pts (xy 139.7 33.02) (xy 196.85 33.02))
     (stroke (width 0) (type dash))
   )
@@
     (stroke (width 0) (type default))
   )
-  (polyline (pts (xy 198.12 12.7) (xy 198.12 33.02))
+  (polyline (pts (xy 196.85 12.7) (xy 196.85 33.02))
     (stroke (width 0) (type dash))
   )
@@
       (effects (font (size 1.27 1.27)))
     )
-    (property "Value" "1k" (at 36.83 77.47 90)
+    (property "Value" "DNP" (at 36.83 77.47 90)
       (effects (font (size 0.8 0.8)))
     )
@@
       (effects (font (size 1.27 1.27)))
     )
-    (property "Value" "27pF" (at 21.59 83.82 90)
+    (property "Value" "22pF" (at 21.59 83.82 90)
       (effects (font (size 1.27 1.27)))
     )
@@
       (effects (font (size 1.27 1.27)))
     )
-    (property "Value" "27pF" (at 21.5963 66.04 90)
-      (effects (font (size 1.27 1.27)))
-    )
+    (property "Value" "22pF" (at 21.5963 66.04 90)
+      (effects (font (size 1.27 1.27)))
+    )
